File: EMUZ80_RP2350B.kicad_pcb (KiCad board)
At the start: 2 copper layers, 99.1 x 75.6 mm, 18 parts, among them J1 SBC8080BUS_2, J4 Conn_01x08_Pin, U1 Z80CPU, U2 RB2350B_Core_Board_for_EMUZ80

Commit message: main: Rev001 almost be ready
Connections:
- U1 pad 28: /RFSH -> unconnected-(U1-~{RFSH}-Pad28)
Routing:
- net /A4: track 139.0 -> 88.5 mm, vias 4 -> 0
- net /A5: track 135.7 -> 92.4 mm, vias 4 -> 2
- net /A6: track 133.9 -> 95.4 mm, vias 4 -> 2
- net /A7: track 131.7 -> 100.8 mm, vias 4 -> 2
- net /A8: track 128.2 -> 102.6 mm, vias 4 -> 2
- net /A12: track 130.9 -> 110.5 mm, vias 4 -> 2
- net /A9: track 130.1 -> 111.3 mm, vias 6 -> 4
- net /A3: track 144.5 -> 127.3 mm, vias 4 -> 5
- net /A2: track 147.5 -> 130.7 mm, vias 5 -> 4
- net /A1: track 150.7 -> 134.4 mm
- net /A11: track 131.1 -> 115.0 mm
- net /A0: track 153.0 -> 137.4 mm
- net /A10: track 128.9 -> 116.5 mm, vias 5 -> 4
- net Net-(J4-Pin_4): track 43.6 -> 46.1 mm
- net /D1: track 58.9 -> 61.3 mm
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Other:
- board text removed: "29"
- board text removed: "3V3"
