File: EMUZ80_RP2350B.kicad_sch (KiCad schematic)
At the start: 14 parts, among them J1 SBC8080BUS_2, J4 Conn_01x08_Pin, U1 Z80CPU, U2 RB2350B_Core_Board_for_EMUZ80

Commit message: main: Rev001 almost be ready
Parts:
- U2: footprint (none) -> local-f:RB2350B_Core_Board
Connections:
- net RFSH: no longer U1.28 (~{RFSH})
Changed lines of the file:
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@@
 	)
 	(no_connect
-		(at 194.31 132.08)
+		(at 359.41 137.16)
 	)
 	(no_connect
@@
 	(wire
 		(pts
-			(xy 198.12 132.08) (xy 198.12 137.16)
-		)
-		(stroke
-			(width 0)
-			(type default)
-		)
-	)
-	(wire
-		(pts
 			(xy 243.84 182.88) (xy 243.84 119.38)
 		)
@@
 	(wire
 		(pts
-			(xy 62.23 60.96) (xy 73.66 60.96)
+			(xy 359.41 137.16) (xy 365.76 137.16)
 		)
 		(stroke
@@
 	(wire
 		(pts
-			(xy 109.22 86.36) (xy 322.58 86.36)
+			(xy 62.23 60.96) (xy 73.66 60.96)
 		)
 		(stroke
@@
 	(wire
 		(pts
-			(xy 327.66 165.1) (xy 327.66 76.2)
+			(xy 109.22 86.36) (xy 322.58 86.36)
 		)
 		(stroke
@@
 	(wire
 		(pts
-			(xy 109.22 35.56) (xy 254 35.56)
+			(xy 327.66 165.1) (xy 327.66 76.2)
 		)
 		(stroke
@@
 	(wire
 		(pts
-			(xy 204.47 121.92) (xy 365.76 121.92)
+			(xy 109.22 35.56) (xy 254 35.56)
 		)
 		(stroke
@@
 	(wire
 		(pts
-			(xy 109.22 83.82) (xy 228.6 83.82)
+			(xy 204.47 121.92) (xy 365.76 121.92)
 		)
 		(stroke
@@
 	(wire
 		(pts
-			(xy 264.16 198.12) (xy 271.78 198.12)
+			(xy 109.22 83.82) (xy 228.6 83.82)
 		)
 		(stroke
@@
 	(wire
 		(pts
-			(xy 198.12 137.16) (xy 365.76 137.16)
+			(xy 264.16 198.12) (xy 271.78 198.12)
 		)
 		(stroke
@@
 	(wire
 		(pts
-			(xy 194.31 132.08) (xy 198.12 132.08)
-		)
-		(stroke
-			(width 0)
-			(type default)
-		)
-	)
-	(wire
-		(pts
 			(xy 109.22 50.8) (xy 261.62 50.8)
 		)
@@
 		)
 	)
-	(label "RFSH"
-		(at 195.58 132.08 0)
-		(effects
-			(font
-				(size 1.27 1.27)
-			)
-			(justify left bottom)
-		)
-	)
 	(label "RD"
 		(at 195.58 101.6 0)
@@
 			)
 		)
-		(property "Footprint" ""
+		(property "Footprint" "local-f:RB2350B_Core_Board"
 			(at 68.58 43.18 0)
 			(effects
